File: PanelLDR/PanelLDR.kicad_pcb (KiCad board)
At the start: 2 copper layers, 45 x 30 mm, 3 parts, among them J1 Conn_01x03, J2 Conn_01x08, J3 Conn_01x03

Commit message: Placas Terminadas
Parts:
- moved J1 10.7 mm to (198.0, 56.5)
- moved J3 10.7 mm to (198.0, 68.6)
Routing:
- net +3.3V: track 75.6 -> 91.9 mm
- net LDR_ID: track 13.8 -> 24.5 mm
- net LDR_SD: track 14.4 -> 25.1 mm
- net LDR_II: track 46.3 -> 56.5 mm
- net LDR_SI: track 48.1 -> 57.8 mm
Other:
- board size 45 x 30 mm -> 55 x 26 mm
