File: SolarTracker/SolarTracker.kicad_pcb (KiCad board)
At the start: 2 copper layers, 90 x 65 mm, 60 parts, among them J1 VIN, J2 MOTOR A, J3 LDR-S, J4 LDR-I, J5 MOTOR B, J6 OLED, J7 JOYSTICK, J8 V_MOTOR, U1 ESP32_DevKit_V1_DOIT, U2 LM7805_TO220

Commit message: Placas Terminadas
Parts:
- removed the C3 at (139.1, 66.7)
- removed the D1 at (142.9, 80.0)
- removed the D2 at (125.7, 76.2)
- removed the J8 at (90.2, 66.7)
- removed the R1 at (125.7, 72.4)
- removed the REF** at (25.4, 177.9)
- removed U2: LM7805_TO220, Package_TO_SOT_THT:TO-220-3_Vertical
- removed kibuzzard-67F1ECE8: G***, kibuzzard-67F1ECE8
- removed kibuzzard-67F1ECF6: G***, kibuzzard-67F1ECF6
- removed kibuzzard-67F1ED07: G***, kibuzzard-67F1ED07
- added J2: V_MOTOR, TerminalBlock_Phoenix:TerminalBlock_Phoenix_MKDS-1,5-2-5.08_1x02_P5.08mm_Horizontal, F.Cu at (104.1, 66.5)
- added kibuzzard-67F2E706: G***, kibuzzard-67F2E706, F.Cu at (139.0, 65.0)
- added kibuzzard-67F2E713: G***, kibuzzard-67F2E713, F.Cu at (139.0, 70.0)
- J1: value VIN -> Barrel_Jack_Switch; footprint TerminalBlock_Phoenix:TerminalBlock_Phoenix_MKDS-1,5-2-5.08_1x02_P5.08mm_Horizontal -> Connector_BarrelJack:BarrelJack_Horizontal
- moved J1 17.5 mm to (87.0, 70.0), turned to -90 degrees
- renumbered C4 to C3, D3 to D1, D4 to D2, J2 to J3, J3 to J4, J4 to J5, J5 to J6, J6 to J7, J7 to J8, R2 to R1, R3 to R2, R4 to R3, R5 to R4, R6 to R5, R7 to R6
Connections:
- J1 pad 1: GND -> VCC
- J1 pad 2: VCC -> GND
- U1 pad 17: unconnected-(U1-GND-Pad17) -> GND
Routing:
- net VCC: track 83.0 -> 46.2 mm
- net Net-(D2-A) (its old number): track 13.1 -> 0.00 mm
- net Net-(D1-A) (its old number): track 10.9 -> 0.00 mm
- net GND: track 65.7 -> 61.1 mm, vias 14 -> 12
- net +5V: track 104.4 -> 100.9 mm
